File: rf_front_lf.brd (EAGLE design)
At the start: 67.3 x 74.9 mm, 112 parts, among them CON1 RF_IN, CON2 PLL_OUT, IC1 RF_AMP, IC2 STW81200, IC3 ADL5380, IC4 TAR5SB33, IC5 7805, J1 SHORT, J2 EXT5V, J3 CS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

Commit message: 発注
Parts:
- removed C53: 4.7n, my_rcl:1608
- removed R19, R20: 1k, my_rcl:1608
- added L10, L11: 150nH, my_rcl:1608
- added TR1: ETC1-1-13, my_rcl:ETC1-1-13
- C25, C26, C27, C28: value 100p -> 1000p
- C52: value 0.1u -> 4.7n
- D1: value LOCK -> PWR
- D2: value PWR -> LOCK
- IC3: value ADL5380 -> ADL5387
- R11: value DNP -> 25
- R17, R18: value 25 -> 1k
- moved C52 36.2 mm to (52.4, 17.8), turned to 0 degrees
- moved R18 24.0 mm to (47.0, 47.6), turned to 270 degrees
- moved R17 24.0 mm to (44.5, 47.6), turned to 270 degrees
- moved C25 14.5 mm to (34.6, 25.2), turned to 0 degrees
- moved R6 14.5 mm to (31.1, 25.2)
- moved C28 13.5 mm to (21.0, 27.6)
- moved R12 12.3 mm to (26.2, 21.6), turned to 90 degrees
- moved R11 12.3 mm to (31.1, 27.1), turned to 180 degrees
- moved C40 7.05 mm to (21.6, 34.3), turned to 90 degrees
- moved FB2 6.82 mm to (19.4, 34.3)
- moved C47 4.77 mm to (23.8, 32.7), turned to 90 degrees
- moved C27 4.18 mm to (21.0, 25.7), turned to 0 degrees
- moved C51 3.13 mm to (24.1, 21.6), turned to 270 degrees
- moved C43 2.93 mm to (28.3, 21.6), turned to 270 degrees
- moved D1 2.86 mm to (44.5, 44.1)
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Connections:
- removed net MIX_ADJ: IC3.19, R11.1, R12.2
- new net N$38: C26.1, R11.1
- new net N$39: D2.K, R18.2
- net +5V: now also D1.A; no longer D2.A
- net GND: now also IC3.10, IC3.12, IC3.24, L10.1, L11.1, R17.1, R18.1, TR1.1, TR1.4; no longer C27.2, C53.2, IC3.1, IC3.14, IC3.17, IC3.18, IC3.5, IC3.8, R19.1, R20.1
- net MIX_IN: now also IC3.13; no longer IC3.4
- net MIX_IP: now also IC3.14; no longer IC3.3
- net MIX_RFIN: now also TR1.2; no longer R6.2
- net N$17: now also C27.1, TR1.3; no longer C26.1, R17.1
- net N$18: now also TR1.5; no longer R18.1
- net N$20: now also IC3.9, R11.2; no longer C27.1, IC3.21
- net N$34: now also D1.K; no longer IC3.9
- net N$35: now also IC3.3, R12.2; no longer IC3.10, R18.2
- net N$36: now also IC3.8, R6.2; no longer D2.K, R20.2
- net N$37: now also C25.1, R6.1; no longer D1.K, R19.2
- net N$4: now also C27.2, IC3.22, L10.2; no longer C25.2, R6.1
- net N$8: now also C28.2, IC3.21, L11.2; no longer C25.1, IC3.22
- net PLL_ICP: now also C52.1; no longer C53.1
- net PLL_OUT2N: now also C26.2; no longer C28.2
- net PLL_OUT2P: now also C25.2; no longer C26.2
- net PLL_SPI_MISO: now also D2.A; no longer D1.A
- net VCC_MIX: now also IC3.1, IC3.17, IC3.18, IC3.19, IC3.4, IC3.5; no longer C52.1, IC3.13, IC3.24, R11.2
Routing:
- net MIX_IP: track 23.5 -> 15.3 mm, vias 2 -> 0
- net MIX_IN: track 27.8 -> 20.0 mm, vias 2 -> 0
- net VCC_MIX: track 48.6 -> 41.8 mm
- net MIX_ADJ: track 6.24 -> 0.00 mm
- net MIX_RFIN: track 4.96 -> 7.92 mm
- net +5V: track 100.2 -> 103.1 mm, vias 3 -> 4
- net PLL_OUT2P: track 11.5 -> 8.69 mm
- net PLL_OUT2N: track 12.8 -> 9.92 mm
- net N$4: track 1.69 -> 4.21 mm
- net N$39: track 0.00 -> 1.69 mm
- net N$38: track 0.00 -> 1.69 mm
- net MIX_QP: track 19.6 -> 21.1 mm, vias 2 -> 0
- net N$8: track 2.69 -> 4.21 mm
- net MIX_QN: track 14.7 -> 16.2 mm, vias 2 -> 0
- net N$18: track 1.69 -> 2.60 mm
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Other:
- board text added: "Spectrum Analyzer LF-Front ver1"
- board text removed: "Spectrum Analyzer HF-Front ver1"
