File: rf_front_lf.sch (EAGLE design)
At the start: 112 parts, among them CON1 RF_IN, CON2 PLL_OUT, IC1 RF_AMP, IC2 STW81200, IC3 ADL5380, IC4 TAR5SB33, IC5 7805, J1 SHORT, J2 EXT5V, J3 CS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

Commit message: 発注
Parts:
- removed C53: 4.7n, my_rcl:C-1608
- removed R19, R20: 1k, my_rcl:R-1608
- added L10, L11: 150nH, my_rcl:L-1608
- added TR1: ETC1-1-13, my_rcl:ETC1-1-13
- C25, C26, C27, C28: value 100p -> 1000p
- C52: value 0.1u -> 4.7n
- D1: value LOCK -> PWR
- D2: value PWR -> LOCK
- IC3: value ADL5380 -> ADL5387; device my_ic:ADL5380 -> my_ic:ADL5387
- R11: value DNP -> 25
- R17, R18: value 25 -> 1k
Connections:
- removed net MIX_ADJ: IC3.ADJ, R11.1, R12.2
- new net N$38: C26.1, R11.1
- new net N$39: D2.K, R18.2
- net +5V: now also D1.A; no longer D2.A
- net GND: now also L10.1, L11.1, R17.1, R18.1, TR1.1, TR1.4; no longer C27.2, C53.2, IC3.ENBL, IC3.GND10, IC3.GND9, R19.1, R20.1
- net MIX_RFIN: now also TR1.2; no longer R6.2
- net N$17: now also C27.1, TR1.3; no longer C26.1, R17.1
- net N$18: now also TR1.5; no longer R18.1
- net N$20: now also IC3.LOIN, R11.2; no longer C27.1, IC3.RFIN
- net N$34: now also D1.K; no longer IC3.LOIP
- net N$35: now also IC3.BIAS, R12.2; no longer IC3.LOIN, R18.2
- net N$36: now also IC3.LOIP, R6.2; no longer D2.K, R20.2
- net N$37: now also C25.1, R6.1; no longer D1.K, R19.2
- net N$4: now also C27.2, IC3.RFIP, L10.2; no longer C25.2, R6.1
- net N$8: now also C28.2, IC3.RFIN, L11.2; no longer C25.1, IC3.RFIP
- net PLL_ICP: now also C52.1; no longer C53.1
- net PLL_OUT1_PD: now also IC2.PDREF1; no longer IC2.PDRF1
- net PLL_OUT2N: now also C26.2; no longer C28.2
- net PLL_OUT2P: now also C25.2; no longer C26.2
- net PLL_OUT2_PD: now also IC2.PDREF2; no longer IC2.PDRF2
- net PLL_SPI_MISO: now also D2.A; no longer D1.A
- net VCC_MIX: now also IC3.VCC4, IC3.VCC5, IC3.VCC6, IC3.VCC7; no longer C52.1, R11.2
Other:
- moved on the sheet: C25, C26, C27, C28, C52, D1, D2, IC3, R11, R12, R17, R18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
