File: SA.sch (EAGLE design)
At the start: 171 parts, among them CON1 RF_IN, CON2 PLL_OUT, CON3 SWD_CON, CON4 USB-C, IC1 RF_AMP, IC10 MCP6D11, IC11 MCP6D11, IC12 TAR5SB33, IC2 STW81200, IC3 ADL5380, IC4 TAR5SB33, IC5 STM32G431KB, IC6 SKY13453, IC7 NJG1809, IC8 SKY13453, IC9 NJG1809, J1 HW_PD, T1 X4B40L1, X1 25MHz, X2 25MHz, X3 12MHz

Commit message: ほぼ完成
Parts:
- removed R2: 10, my_rcl:R-1608
- added C82: 0.1u, my_rcl:C-1608
- added C83: 100p, my_rcl:C-1608
- added L10: 47nH, my_rcl:L-1005
- added R40: 10k, my_rcl:R-1608
- added SW1: BOOT0, my_rcl:SW-SMD
- C25, C27, C55: value 22p -> 100p; device my_rcl:C-1608 -> my_rcl:C-1005
- C26, C28, C3, C31, C32, C54, C56, C57: device my_rcl:C-1608 -> my_rcl:C-1005
- C41: value 0.01u -> 1u
- C44: value 1u -> 10n
- DR1, DR2, DR3, DR4: value HOLE-3.2 -> HOLE-3.2-CON; device my_connector:HOLE-3.2 -> my_connector:HOLE-3.2-CON
- FIL1: value 5515LP15A730 -> 5515LP15A0730001E
- FIL3: device my_rcl:RF-FILTER-1608-TDK2 -> my_rcl:RF-FILTER-1608-TDK3
- FIL6: value DEA162025LT-5046C1 -> DEA160960LT-5059A1
- FIL8: value DEA162300HT-8047A1 -> DEA162400HT-8053A1; device my_rcl:RF-FILTER-1608-TDK3 -> my_rcl:RF-FILTER-1608-TDK
- IC1: value RF_AMP -> ADL5611
- L1: value 150nH -> 47nH; device my_rcl:L-1608 -> my_rcl:L-1005
- L2, L3, L4, L5, L6, L7, L8, L9: value 10u -> 10uH
- R1: value DNP -> 50; device my_rcl:R-1608 -> my_rcl:R-1005
- R13, R14, R17, R18: device my_rcl:R-1608 -> my_rcl:R-1005
Connections:
- net N$23 renamed PLL_OUT
- removed net N$19: L1.1, R2.1
- new net N$23: L10.2, R1.2
- new net ST_BOOT0: IC5.BOOT0, R40.2, SW1.2
- new net ST_NRST: C82.1, IC5.NRST
- net +3V3: now also IC10G$1.EN, IC11G$1.EN
- net +3V3D: now also SW1.1
- net FILTER_IN: now also FIL1.IN; no longer FIL1.RF1
- net GND: now also C82.2, C83.2, R40.1; no longer IC10G$1.EN, IC11G$1.EN, IC5.BOOT0
- net MIX_IN: now also R8.1; no longer C61.1
- net MIX_IP: now also R7.1; no longer C60.1
- net MIX_QN: now also R10.1; no longer C63.1
- net MIX_QP: now also R9.1; no longer C62.1
- net N$32: now also C60.2; no longer R7.2
- net N$33: now also C61.2; no longer R8.2
- net N$38: now also FIL1.OUT; no longer FIL1.RF2
- net N$45: now also FIL2.IN; no longer FIL2.RF1
- net N$46: now also FIL4.IN; no longer FIL4.RF1
- net N$47: now also FIL3.IN; no longer FIL3.RF1
- net N$48: now also FIL4.OUT, FIL5.IN; no longer FIL4.RF2, FIL5.RF1
- net N$49: now also FIL6.IN; no longer FIL6.RF1
- net N$50: now also FIL6.OUT, FIL7.IN; no longer FIL6.RF2, FIL7.RF1
- net N$51: now also FIL3.OUT, FIL8.IN; no longer FIL3.RF2, FIL8.RF1
- net N$52: now also FIL2.OUT; no longer FIL2.RF2
- net N$53: now also FIL8.OUT; no longer FIL8.RF2
- net N$54: now also FIL5.OUT; no longer FIL5.RF2
- net N$55: now also FIL7.OUT; no longer FIL7.RF2
- net N$58: now also C60.1, R7.2; no longer C60.2, R7.1
- net N$59: now also C61.1, R8.2; no longer C61.2, R8.1
- net N$60: now also C62.1, R9.2; no longer C62.2, R9.1
- net N$61: now also C63.1, R10.2; no longer C63.2, R10.1
- net N$7: now also C62.2; no longer R9.2
- net N$9: now also C63.2; no longer R10.2
- net RF_IN: now also L10.1; no longer R1.2
- net VCC_HFAMP: now also C83.1, L1.1; no longer R2.2
Other:
- note added: "LPF 1.5GHz"
- moved on the sheet: C3, C54, C55, C56, C57, C60, C61, C62, C63, CON1, FIL2, FIL4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

Commit message: OK
Parts:
- added D3: LED, my_rcl:LED-SMD1608
- added R2: 1k, my_rcl:R-1608
- added TP1: +5V, my_connector:TESTPIN
- added TP2: GND, my_connector:TESTPIN
- IC5: value STM32G431KB -> STM32G431K
Connections:
- new net N$19: IC5.PB0, R30.1
- new net N$73: IC5.PA4, R2.1
- net +5V: now also TP1.1
- net GND: now also D3.K, TP2.1
- net N$24: now also R31.1; no longer R30.1
- net N$25: now also R32.1; no longer R31.1
- net N$27: now also R33.1; no longer R32.1
- net N$28: now also D3.A, R2.2; no longer IC5.PA4, R33.1
Other:
- moved on the sheet: C21, C37, C38, C59, C69, C70, C71, C72, C73, C74, C75, IC12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

Commit message: STw81200
Parts:
- removed C28: 100p, my_rcl:C-1005
- removed L1: 47nH, my_rcl:L-1005
- removed L4: 10uH, my_rcl:L-2012
- removed X2: 25MHz, my_rcl:CRYSTAL2
- added ATT1: 3dB, my_ic:RF-ATT
- added C84: 10p, my_rcl:C-1608
- added C85, C86, C88, C89: 0.1u, my_rcl:C-1608
- added C87: 10u, my_rcl:C-2012
- added CON5: USB-C, my_connector:USB-C
- added FIL9: DEA160787LT-5032A1, my_rcl:RF-FILTER-1608-TDK2
- added IC13: TLV3542, my_ic:OPA-2-SOP
- added IC14, IC15: TAR5SB33, my_ic:TAR5SB33
- added IC16: STM32G431K, my_ic:STM32G431KB
- added L11, L12: 10uH, my_rcl:L-2012
- added R41, R42, R44: 1k, my_rcl:R-1608
- added R43: 10k, my_rcl:R-1608
- added R45, R46, R47, R48: 39, my_rcl:R-1608
- added R49, R50: 5.1k, my_rcl:R-1608
- added TP3, TP5, TP6, TP7, TP8: GND, my_connector:TESTPIN
- added TP4: +5V, my_connector:TESTPIN
- C1: device my_rcl:C-1608 -> my_rcl:C-2012
- C13: value 47n -> 4.7n
- C14: value 10u -> 47n
- C15, C18: value 0.1u -> 100p; device my_rcl:C-1608 -> my_rcl:C-1005RF
- C16, C46, C51, C7, C82: value 0.1u -> 10u; device my_rcl:C-1608 -> my_rcl:C-2012
- C19, C20, C62, C63, C8: value 10u -> 0.1u
- C22: value 10p -> 100p; device my_rcl:C-1608 -> my_rcl:C-1005RF
- C23: value 10p -> 10u; device my_rcl:C-1608 -> my_rcl:C-2012
- C24: value DNP -> 10u; device my_rcl:C-1608 -> my_rcl:C-2012
- C25, C26: device my_rcl:C-1005 -> my_rcl:C-1005RF
- C27: value 100p -> 10p; device my_rcl:C-1005 -> my_rcl:C-1608
- C29: value 1000p -> DNP
- C3: value 22p -> 0.1u; device my_rcl:C-1005 -> my_rcl:C-1608
- C30, C35, C36: value 1000p -> 100p; device my_rcl:C-1608 -> my_rcl:C-1005RF
- C31, C32: value 100p -> 10u; device my_rcl:C-1005 -> my_rcl:C-1608
- C33: value 3300p -> 10u
- C34: value 470p -> 10u
- C37: value 1u -> 100p; device my_rcl:C-1608 -> my_rcl:C-1005RF
- C38: value 10u -> 100p; device my_rcl:C-2012 -> my_rcl:C-1005RF
- C39, C40: value 10u -> 1000p; device my_rcl:C-2012 -> my_rcl:C-1608
- C41: value 1u -> 3300p
- C42: value 0.1u -> 3300p
- C43: value 0.1u -> 1000p
- C44: value 10n -> 1000p
- C45: value 10u -> 1n; device my_rcl:C-1608 -> my_rcl:C-1005
- C47, C75: value 0.1u -> 1u
- C48, C49: value 22p -> 1u
- C50: value 22p -> 10u; device my_rcl:C-1608 -> my_rcl:C-3216
- C52, C81: value 1u -> 0.1u
- C53: value 4.7n -> 10n
- C54, C55: value 100p -> 0.01u; device my_rcl:C-1005 -> my_rcl:C-1608
- C56: value 100p -> 10u; device my_rcl:C-1005 -> my_rcl:C-2012
- C57: value 100p -> 0.1u; device my_rcl:C-1005 -> my_rcl:C-1608
- C58: value 22p -> 0.1u
- C59: value 1u -> 100p; device my_rcl:C-1608 -> my_rcl:C-1005
- C60, C61: value 10u -> 0.01u
- C64: value 0.01u -> 1n; device my_rcl:C-1608 -> my_rcl:C-1005
- C65, C66, C67: value 0.01u -> 22p
- C68: value 0.1u -> 22p
- C69: value 10u -> 1n; device my_rcl:C-2012 -> my_rcl:C-1005
- C71: value 0.1u -> 1n; device my_rcl:C-1608 -> my_rcl:C-1005
- C77: value 10p -> 0.1u
- C78: value 10p -> 1u
- C79: device my_rcl:C-2012 -> my_rcl:C-1608
- C80: value 10u -> 10p; device my_rcl:C-3216 -> my_rcl:C-1608
- C83: value 100p -> 0.1u
- C9: value 0.1u -> 22p; device my_rcl:C-1608 -> my_rcl:C-1005RF
- CON1: value RF_IN -> DM_L
- CON2: value PLL_OUT -> RF_IN
- CON3: value SWD_CON -> PLL_OUT; device my_connector:SWD_CON -> my_connector:SMA-142-0701-801
- CON4: value USB-C -> SWD_CON; device my_connector:USB-C -> my_connector:SWD_CON
- D1: value LOCK -> PWR
- D2: value PWR -> LED
- D3: value LED -> LOCK
- FB1, FB2, FB3, FB4, FB5: device my_rcl:FB -> my_rcl:FB-1608FB
- FB7: value FB -> (none)
- FIL5: value DEA162025LT-5046C1 -> DEA160960LT-5059A1
- FIL6: value DEA160960LT-5059A1 -> DEA165150HT-8025C2
- FIL7: value DEA160787LT-5032A1 -> DEA162400HT-8053A1; device my_rcl:RF-FILTER-1608-TDK2 -> my_rcl:RF-FILTER-1608-TDK
- FIL8: value DEA162400HT-8053A1 -> DEA162025LT-5046C1
- IC1: value ADL5611 -> QPC6044; device my_ic:RF_AMP -> my_ic:QPC6044
- IC10, IC11: value MCP6D11 -> SN74LVC1G66; device my_ic:OPA-DIFF-MSOP -> my_ic:SN74LVC1G66
- IC12: value TAR5SB33 -> TLV3542; device my_ic:TAR5SB33 -> my_ic:OPA-2-SOP
- IC2: value STW81200 -> SKY13453; device my_ic:STW81200 -> my_ic:SKY13453
- IC3: value ADL5380 -> STW81200; device my_ic:ADL5380 -> my_ic:STW81200
- IC4: value TAR5SB33 -> ADL5611; device my_ic:TAR5SB33 -> my_ic:RF_AMP
- IC5: value STM32G431K -> SKY13453; device my_ic:STM32G431KB -> my_ic:SKY13453
- IC6: value SKY13453 -> QPC6044; device my_ic:SKY13453 -> my_ic:QPC6044
- IC7: value NJG1809 -> ADL5380; device my_ic:NJG1809 -> my_ic:ADL5380
- IC8: value SKY13453 -> MCP6D11; device my_ic:SKY13453 -> my_ic:OPA-DIFF-MSOP
- IC9: value NJG1809 -> MCP6D11; device my_ic:NJG1809 -> my_ic:OPA-DIFF-MSOP
- L10: value 47nH -> 10uH; device my_rcl:L-1005 -> my_rcl:L-2012
- L2: value 10uH -> 47nH; device my_rcl:L-2012 -> my_rcl:L-1005RF
- L3: value 10uH -> 47nH; device my_rcl:L-2012 -> my_rcl:L-1608
- R1: device my_rcl:R-1005 -> my_rcl:R-1005RF
- R10, R7, R8, R9: value 25 -> 360
- R11, R12: value DNP -> 25
- R13: value 50 -> 25; device my_rcl:R-1005 -> my_rcl:R-1608
- R14: value DNP -> 25; device my_rcl:R-1005 -> my_rcl:R-1608
- R15: value 120 -> 25; device my_rcl:R-1608 -> my_rcl:R-1005RF
- R16: value 120 -> 10k
- R17: value 25 -> 10k; device my_rcl:R-1005 -> my_rcl:R-1608-3
- R18: value 25 -> 10k; device my_rcl:R-1005 -> my_rcl:R-1608
- R19: value 1k -> 10k; device my_rcl:R-1608 -> my_rcl:R-1608-3
- R2: value 1k -> 50; device my_rcl:R-1608 -> my_rcl:R-1005RF
- R20: value 1k -> 25; device my_rcl:R-1608 -> my_rcl:R-1005RF
- R21, R22: value 10k -> DNP
- R23, R24: value 360 -> 120
- R25, R26: value 10k -> 1k
- R27: value 360 -> 47; device my_rcl:R-1608 -> my_rcl:R-1608-3
- R28, R29: value 10k -> 47; device my_rcl:R-1608 -> my_rcl:R-1608-3
- R30: value 39 -> 47; device my_rcl:R-1608J -> my_rcl:R-1608-3
- R31, R32, R33: value 39 -> 1k; device my_rcl:R-1608J -> my_rcl:R-1608-3
- R34: value 5.1k -> 1k; device my_rcl:R-1608 -> my_rcl:R-1608-3
- R35: value 5.1k -> 39
- R39: value 39 -> 1.5k
- R40: value 10k -> 1.5k
- R6: value 360 -> 50; device my_rcl:R-1608 -> my_rcl:R-1005RF
Connections:
- removed net N$55: FIL7.OUT, IC9.P3
- new net DUMMY_LOAD: CON1.SIG, R1.2
- new net N$74: IC12G$1.-IN, R27.2, R31.2
- new net N$75: IC12G$2.+IN, IC8G$1.+OUT, R17.2
- new net N$76: IC12G$1.OUT, R31.1, R35.1
- new net N$77: IC13G$2.+IN, IC9G$1.+OUT, R19.2
- new net N$78: IC13G$2.OUT, R34.1, R38.1
- new net N$79: IC12G$2.OUT, R32.1, R36.1
- new net N$80: IC13G$2.-IN, R30.2, R34.2
- new net N$81: IC13G$1.OUT, R33.1, R37.1
- new net N$82: ATT1.SIG2, C25.2
- new net N$83: IC10.B, R25.1, R28.1
- new net N$84: IC10.A, R25.2, R27.1
- new net N$85: IC11.B, R26.1, R30.1
- new net N$86: IC11.A, R26.2, R29.1
- new net N$87: FIL3.IN, IC1.P3
- new net PGA_SW: IC10.S, IC11.S, IC16.PA4, R44.1
- net +3V3: now also C73.1, C77.1, C87.1, FB5.1, IC12G$3.V+, IC13G$3.V+, IC15.VOUT, R39.2; no longer C38.1, C74.1, C75.1, FB7.1, IC10G$1.EN, IC10G$2.V+, IC11G$1.EN, IC11G$2.V+, IC4.VOUT, R28.2
- net +3V3D: now also C82.1, C86.1, C88.1, C89.1, FB7.1, IC14.VOUT, IC16.VDDA, IC16.VDD_1, IC16.VDD_2; no longer C69.1, C71.1, C72.1, C73.1, FB5.1, IC12.VOUT, IC5.VDDA, IC5.VDD_1, IC5.VDD_2
- net +5V: now also C50.1, C56.1, C72.1, C75.1, C76.1, C78.1, D1.A, IC10.VCC, IC11.VCC, IC14.CONTROL, IC14.VIN, IC15.CONTROL, IC15.VIN, IC8G$2.EN, IC8G$2.V+, IC9G$2.EN, IC9G$2.V+, TP4.1; no longer C37.1, C59.1, C79.1, C80.1, D2.A, IC12.CONTROL, IC12.VIN, IC4.CONTROL, IC4.VIN
- net ADC_IN: now also C65.2, IC16.PA2, R35.2; no longer C49.2, IC5.PA2, R36.2
- net ADC_IP: now also C66.1, IC16.PA3, R36.2; no longer C48.1, IC5.PA3, R37.2
- net ADC_QN: now also C67.2, IC16.PA0, R37.2; no longer C50.2, IC5.PA0, R38.2
- net ADC_QP: now also C68.1, IC16.PA1, R38.2; no longer C58.1, IC5.PA1, R39.2
- net AMP_IN: now also C43.2, L10.2, R8.1; no longer C35.2, L7.2, R15.1
- net AMP_IP: now also C43.1, L9.2, R23.2, R7.1; no longer C35.1, L6.2, R15.2, R6.1
- net AMP_QN: now also C44.2, L12.2, R10.1, R24.1; no longer C36.2, L9.2, R16.1, R27.1
- net AMP_QP: now also C44.1, L11.2, R24.2, R9.1; no longer C36.1, L8.2, R16.2, R24.1
- net FILTER_IN: now also C30.2; no longer C57.2
- net FILTER_OUT: now also IC6.PC; no longer IC9.PC
- net FIL_SW1: now also IC1.CTL1, IC16.PB5; no longer IC5.PB5, IC7.CTL1
- net FIL_SW2: now also IC1.CTL2, IC16.PB4; no longer IC5.PB4, IC7.CTL2
- net FIL_SW3: now also IC16.PA9, IC6.CTL1; no longer IC5.PA9, IC9.CTL1
- net FIL_SW4: now also IC16.PA8, IC6.CTL2; no longer IC5.PA8, IC9.CTL2
- net GND: now also ATT1.GND, C13.2, C20.2, C21.1, C24.1, C27.2, C3.2, C49.2, C50.2, C54.2, C55.2, C56.2, C57.2, C60.2, C61.2, C62.2, C63.2, C65.1, C67.1, C7.2, C84.2, C85.2, C86.2, C87.2, C88.2, C89.2, CON5.GND, CON5.XT, D2.K, FIL9.GND, IC1.CTL3, IC1.VSS, IC10.GND, IC11.GND, IC12G$3.V-, IC13G$3.V-, IC14.GND, IC15.GND, IC16.VSSA, IC16.VSS_1, IC16.VSS_2, IC3.EXTVCO_INN, IC3.EXTVCO_INP, IC3.GND, IC3.PDRF1, IC3.PDRF2, IC3.TEST_SE, IC5.GND, IC6.CTL3, IC6.VSS, IC7.ENBL, IC7.GND@1, IC7.GND@10, IC7.GND@2, IC7.GND@3, IC7.GND@4, IC7.GND@5, IC7.GND@6, IC7.GND@7, IC7.GND@8, IC7.GND@9, IC7.HT, IC8G$2.V-, IC9G$2.V-, R2.1, R22.1, R41.1, R42.1, R43.1, R49.1, R50.1, R6.1, TP3.1, TP5.1, TP6.1, TP7.1, TP8.1; no longer C14.2, C15.2, C18.1, C20.1, C21.2, C22.2, C37.2, C38.2, C39.2, C40.2, C41.2, C42.2, C43.2, C44.2, C49.1, C5.2, C50.1, C65.2, C67.2, C9.2, CON4.XT, D3.K, IC10G$2.V-, IC11G$2.V-, IC12.GND, IC2.EXTVCO_INN, IC2.EXTVCO_INP, IC2.PDRF1, IC2.PDRF2, IC2.TEST_SE, IC3.ENBL, IC3.GND1, IC3.GND10, IC3.GND2, IC3.GND3, IC3.GND4, IC3.GND5, IC3.GND6, IC3.GND7, IC3.GND8, IC3.GND9, IC3.HT, IC5.VSSA, IC5.VSS_1, IC5.VSS_2, IC7.GND, IC8.GND, IC9.GND, R12.1, R13.1, R14.1, R19.1, R20.1, R29.1, R34.1, R35.1, X2.GND
- net MIX_ADJ: now also IC7.ADJ, R21.1, R22.2; no longer IC3.ADJ, R11.1, R12.2
- net MIX_IN: now also IC7.ILO, R12.1; no longer IC3.ILO, R8.1
- net MIX_IP: now also IC7.IHI, R11.1; no longer IC3.IHI, R7.1
- net MIX_QN: now also IC7.QLO, R14.1; no longer IC3.QLO, R10.1
- net MIX_QP: now also IC7.QHI, R13.1; no longer IC3.QHI, R9.1
- net N$1: now also C15.1, IC2.RF2; no longer C54.1, IC8.RF2
- net N$10: now also C42.1, L11.1, L7.2; no longer C34.1, L4.2, L8.1
- net N$11: now also C42.2, L12.1, L8.2; no longer C34.2, L5.2, L9.1
- net N$12: now also IC3.VR; no longer IC2.VR
- net N$13: now also C5.1, IC3.CBYP_4V5; no longer C6.1, IC2.CBYP_4V5
- net N$14: now also C27.1, IC3.REF_CLKN; no longer C22.1, IC2.REF_CLKN, X2.1
- net N$15: now also C6.1, IC3.CBYP; no longer C7.1, IC2.CBYP
- net N$16: now also C29.1, IC3.REF_CLKP; no longer C23.1, C24.1, IC2.REF_CLKP, X2.2
- net N$17: now also C36.1, R15.1; no longer C26.1, R17.1
- net N$18: now also C38.1, R20.1; no longer C28.1, R18.1
- net N$19: now also IC16.PA5, R45.1; no longer IC5.PB0, R30.1
- net N$2: now also C14.2; no longer C13.2
- net N$20: now also C37.1, IC7.RFIN; no longer C27.1, IC3.RFIN
- net N$21: now also C29.2; no longer C24.2
- net N$22: now also C83.1, IC15.BYPASS; no longer C21.1, IC4.BYPASS
- net N$23: now also L2.2, R2.2; no longer L10.2, R1.2
- net N$24: now also IC16.PA6, R46.1; no longer IC5.PA7, R31.1
- net N$25: now also IC16.PA7, R47.1; no longer IC5.PA6, R32.1
- net N$26: now also C26.2, R6.2; no longer C32.2, R13.2
- net N$27: now also IC16.PB0, R48.1; no longer IC5.PA5, R33.1
- net N$28: now also D2.A, R44.2; no longer D3.A, R2.2
- net N$29: now also CON5.CC2, R50.2; no longer CON4.CC2, R34.2
- net N$3: now also C41.1, L5.2, L9.1; no longer C33.1, L2.2, L6.1
- net N$30: now also CON5.CC1, R49.2; no longer CON4.CC1, R35.2
- net N$31: now also IC3.HW_PD; no longer IC2.HW_PD
- net N$32: now also C31.2, C39.1, L5.1; no longer C29.1, C60.2, L2.1
- net N$33: now also C32.2, C39.2, L6.1; no longer C29.2, C61.2, L3.1
- net N$34: now also IC7.LOIP, R15.2; no longer IC3.LOIP, R17.2
- net N$35: now also IC7.LOIN, R20.2; no longer IC3.LOIN, R18.2
- net N$36: now also D1.K, R41.2; no longer D2.K, R20.2
- net N$37: now also D3.K, R42.2; no longer D1.K, R19.2
- net N$38: now also IC1.PC; no longer IC7.PC
- net N$39: now also C18.1, IC2.RF1; no longer C56.1, IC8.RF1
- net N$4: now also C37.2; no longer C27.2
- net N$40: now also C18.2, IC5.RF2; no longer C56.2, IC6.RF2
- net N$41: now also C30.1, IC5.RFC; no longer C57.1, IC6.RFC
- net N$42: now also C9.2, IC2.RFC; no longer C3.2, IC8.RFC
- net N$43: now also C15.2, IC4.IN; no longer C54.2, IC1.IN
- net N$44: now also C22.1, IC4.OUT, L3.2; no longer C55.1, IC1.OUT, L1.2
- net N$45: now also FIL5.IN, IC1.P4; no longer FIL2.IN, IC7.P4
- net N$46: now also IC1.P1; no longer IC7.P3
- net N$47: now also FIL2.IN, IC1.P2; no longer FIL3.IN, IC7.P2
- net N$48: now also FIL8.IN; no longer FIL5.IN
- net N$49: now also FIL6.OUT, IC6.P3; no longer FIL6.IN, IC7.P1
- net N$50: now also FIL5.OUT, FIL9.IN; no longer FIL6.OUT, FIL7.IN
- net N$51: now also FIL7.IN; no longer FIL8.IN
- net N$52: now also FIL7.OUT, IC6.P2; no longer FIL2.OUT, IC9.P2
- net N$53: now also FIL9.OUT, IC6.P1; no longer FIL8.OUT, IC9.P4
- net N$54: now also FIL8.OUT, IC6.P4; no longer FIL5.OUT, IC9.P1
- net N$56: now also C35.2; no longer C25.2
- net N$57: now also C22.2, IC5.RF1; no longer C55.2, IC6.RF1
- net N$58: now also C31.1, R11.2; no longer C60.1, R7.2
- net N$59: now also C32.1, R12.2; no longer C61.1, R8.2
- net N$6: now also C41.2, L10.1, L6.2; no longer C33.2, L3.2, L7.1
- net N$60: now also C33.1, R13.2; no longer C62.1, R9.2
- net N$61: now also C34.1, R14.2; no longer C63.1, R10.2
- net N$62: now also IC8G$1.+IN, R16.1, R7.2; no longer IC10G$1.+IN, R21.1, R6.2
- net N$63: now also IC8G$1.-IN, R17.1, R8.2; no longer IC10G$1.-IN, R22.1, R23.2
- net N$64: now also IC12G$1.+IN, IC8G$1.-OUT, R16.2; no longer IC10G$1.-OUT, R21.2, R36.1
- net N$65: now also IC13G$1.-IN, R29.2, R33.2; no longer IC10G$1.+OUT, R22.2, R37.1
- net N$66: now also IC9G$1.+IN, R18.1, R9.2; no longer IC11G$1.+IN, R24.2, R25.1
- net N$67: now also IC9G$1.-IN, R10.2, R19.1; no longer IC11G$1.-IN, R26.1, R27.2
- net N$68: now also IC12G$2.-IN, R28.2, R32.2; no longer IC11G$1.+OUT, R26.2, R39.1
- net N$69: now also IC13G$1.+IN, IC9G$1.-OUT, R18.2; no longer IC11G$1.-OUT, R25.2, R38.1
- net N$7: now also C33.2, C40.1, L7.1; no longer C30.1, C62.2, L4.1
- net N$70: now also C81.1, IC14.BYPASS; no longer C70.1, IC12.BYPASS
- net N$71: now also C80.1, IC16.PF0/OSC_IN; no longer C78.1, IC5.PF0/OSC_IN
- net N$72: now also C84.1, IC16.PF1_OSC_OUT; no longer C77.1, IC5.PF1_OSC_OUT
- net N$73: now also FIL2.OUT, FIL6.IN; no longer IC5.PA4, R2.1
- net N$8: now also C35.1, IC7.RFIP; no longer C25.1, IC3.RFIP
- net N$9: now also C34.2, C40.2, L8.1; no longer C30.2, C63.2, L5.1
- net PLL_ICP: now also C14.1, IC3.ICP; no longer C53.1, IC2.ICP
- net PLL_OUT: now also ATT1.SIG1, CON3.SIG; no longer C31.2, CON2.SIG, R14.2
- net PLL_OUT1N: now also C26.1, IC3.REF2_OUTN; no longer C32.1, IC2.REF2_OUTN
- net PLL_OUT1P: now also C25.1, IC3.REF2_OUTP; no longer C31.1, IC2.REF2_OUTP
- net PLL_OUT2N: now also C38.2, IC3.REF1_OUTN; no longer C28.2, IC2.REF1_OUTN
- net PLL_OUT2P: now also C36.2, IC3.REF1_OUTP; no longer C26.2, IC2.REF1_OUTP
- net PLL_SPI_CS: now also IC3.LE, R48.2; no longer IC2.LE, R33.2
- net PLL_SPI_MISO: now also D3.A, IC3.SDO, R46.2; no longer D1.A, IC2.SDO, R31.2
- net PLL_SPI_MOSI: now also IC3.SDI, R47.2; no longer IC2.SDI, R30.2
- net PLL_SPI_SCK: now also IC3.SCK, R45.2; no longer IC2.SCK, R32.2
- net PLL_VCTRL: now also IC3.VCTRL; no longer IC2.VCTRL
- net RFIN_SW1: now also IC16.PB6, IC2.VCTL; no longer IC5.PB6, IC8.VCTL
- net RFIN_SW2: now also IC16.PB7, IC5.VCTL; no longer IC5.PB7, IC6.VCTL
- net RF_IN: now also C9.1, CON2.SIG, L2.1; no longer C3.1, CON1.SIG, L10.1
- net ST_BOOT0: now also IC16.BOOT0, R43.2; no longer IC5.BOOT0, R40.2
- net ST_NRST: now also C85.1, IC16.NRST; no longer C82.1, IC5.NRST
- net SWCLK: now also CON4.SWCLK, IC16.PA14/SWCLK; no longer CON3.SWCLK, IC5.PA14/SWCLK
- net SWDIO: now also CON4.SWDIO, IC16.PA13/SWDIO; no longer CON3.SWDIO, IC5.PA13/SWDIO
- net UART_RX: now also CON4.!RST, IC16.PA15; no longer CON3.!RST, IC5.PA15
- net UART_TX: now also CON4.TX, IC16.PB3; no longer CON3.TX, IC5.PB3
- net USB_DM: now also CON5.D-, IC16.PA11; no longer CON4.D-, IC5.PA11
- net USB_DP: now also CON5.D+, IC16.PA12; no longer CON4.D+, IC5.PA12
- net USB_VBUS: now also CON5.VBUS; no longer CON4.VBUS
- net VCC_HFAMP: now also C47.1, C53.1, C59.1, L3.1; no longer C41.1, C44.1, C83.1, L1.1
- net VCC_MIX: now also C46.1, C52.1, C58.1, C63.1, C64.1, C69.1, C71.1, IC7.VCC@1, IC7.VCC@2, IC7.VCC@3, R21.2; no longer C40.1, C43.1, C47.1, C51.1, IC3.VCC1, IC3.VCC2, IC3.VCC3, R11.2
- net VCC_OSC: now also C20.1, C79.1, FB7.2; no longer C17.1, C45.1, FB5.2
- net VCC_RFSW1: now also C49.1, C55.1, C61.1, FB5.2, IC2.VDD, IC5.VDD; no longer C66.1, C67.1, C81.1, FB7.2, IC6.VDD, IC8.VDD
- net VCC_RFSW2: now also C48.1, C54.1, C60.1, IC1.VDD, IC6.VDD; no longer C52.1, C64.1, C65.1, IC7.VDD, IC9.VDD
- net VCOM: now also C70.1, C74.1, IC8G$1.CM, IC9G$1.CM, R39.1, R40.2; no longer C68.1, C76.1, IC10G$1.CM, IC11G$1.CM, R28.1, R29.2
- net VIN_PLL: now also C45.1, C51.1, C57.1, C62.1, IC3.VIN_LDO_4V5, IC3.VIN_LDO_REF, IC3.VIN_LDO_RF_DIG, IC3.VIN_LDO_VCO; no longer C39.1, C42.1, C46.1, IC2.VIN_LDO_4V5, IC2.VIN_LDO_REF, IC2.VIN_LDO_RF_DIG, IC2.VIN_LDO_VCO
- net VREG_4V5: now also C3.1, C5.2, IC3.VCC_CPOUT, IC3.VCC_RFOUT, IC3.VCC_VCO_CORE, IC3.VREG_4V5; no longer C5.1, C6.2, IC2.VCC_CPOUT, IC2.VCC_RFOUT, IC2.VCC_VCO_CORE, IC2.VREG_4V5
- net VREG_DIG: now also C21.2, C24.2, IC3.VDD_DSM_NDIV, IC3.VREG_DIG; no longer C18.2, C20.2, IC2.VDD_DSM_NDIV, IC2.VREG_DIG
- net VREG_REF: now also C23.1, IC3.VDD_PFD, IC3.VREG_REF; no longer C16.1, IC2.VDD_PFD, IC2.VREG_REF
- net VREG_RF: now also C16.1, C17.1, IC3.VREG_RF; no longer C14.1, C15.1, IC2.VREG_RF
- net VREG_VCO: now also C6.2, C7.1, IC3.VDD_CP, IC3.VREG_VCO; no longer C7.2, C9.1, IC2.VDD_CP, IC2.VREG_VCO
Other:
- moved on the sheet: C13, C14, C15, C16, C17, C18, C19, C20, C21, C22, C23, C24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

Commit message: PLLをLMX2572に
Parts:
- removed ATT1: 3dB, my_ic:RF-ATT
- removed C88, C89: 0.1u, my_rcl:C-1608
- removed FB7: (no value), my_rcl:FB
- removed J1: HW_PD, my_rcl:SJ-1608
- removed L12: 10uH, my_rcl:L-2012
- added C28: 0.1u, my_rcl:C-1608
- added IC17: TAR5SB33, my_ic:TAR5SB33
- added IC18: STM32G431K, my_ic:STM32G431KB
- added L1: 47nH, my_rcl:L-1005RF
- added L4: 10uH, my_rcl:L-2012
- added R51, R52: 5.1k, my_rcl:R-1608
- added TP9: GND, my_connector:TESTPIN
- C10: value 680p -> 120n
- C11: value 4.7n -> 10n
- C13: value 4.7n -> 10u
- C14: value 47n -> 100p; device my_rcl:C-1608 -> my_rcl:C-1005RF
- C16: device my_rcl:C-2012 -> my_rcl:C-1608
- C19, C70, C73, C74, C8: value 0.1u -> 1u
- C21: value 0.1u -> 100p; device my_rcl:C-1608 -> my_rcl:C-1005RF
- C23, C24, C82: value 10u -> 0.1u; device my_rcl:C-2012 -> my_rcl:C-1608
- C25: value 100p -> 0.1u; device my_rcl:C-1005RF -> my_rcl:C-1608
- C27, C80: value 10p -> 0.1u
- C29: value DNP -> 10u
- C3, C4: value 0.1u -> 1n
- C30: value 100p -> 10u; device my_rcl:C-1005RF -> my_rcl:C-1608
- C33, C34: value 10u -> 100p; device my_rcl:C-1608 -> my_rcl:C-1005RF
- C37, C38: value 100p -> 1000p; device my_rcl:C-1005RF -> my_rcl:C-1608
- C39, C40: value 1000p -> 3300p
- C41, C42: value 3300p -> 1000p
- C43: value 1000p -> 10u; device my_rcl:C-1608 -> my_rcl:C-2012
- C44: value 1000p -> 1u
- C45: value 1n -> 1u; device my_rcl:C-1005 -> my_rcl:C-1608
- C46, C51, C87: value 10u -> 1u; device my_rcl:C-2012 -> my_rcl:C-1608
- C47: value 1u -> 10u; device my_rcl:C-1608 -> my_rcl:C-3216
- C48: value 1u -> 0.1u
- C49: value 1u -> 10n
- C5: value 0.1u -> 22p; device my_rcl:C-1608 -> my_rcl:C-1005RF
- C50: value 10u -> 0.01u; device my_rcl:C-3216 -> my_rcl:C-1608
- C52, C77, C85: value 0.1u -> 10u; device my_rcl:C-1608 -> my_rcl:C-2012
- C53: value 10n -> 0.1u
- C54: value 0.01u -> 100p; device my_rcl:C-1608 -> my_rcl:C-1005
- C56: value 10u -> 0.01u; device my_rcl:C-2012 -> my_rcl:C-1608
- C58: value 0.1u -> 0.01u
- C59: value 100p -> 1n
- C6: value 0.1u -> 0.47u
- C60, C61: value 0.01u -> 22p
- C62, C63: value 0.1u -> 22p
- C65, C67, C68: value 22p -> 0.1u
- C66: value 22p -> 1n; device my_rcl:C-1608 -> my_rcl:C-1005
- C69, C71: value 1n -> 0.1u; device my_rcl:C-1005 -> my_rcl:C-1608
- C7: value 10u -> 1.5n; device my_rcl:C-2012 -> my_rcl:C-1608
- C75, C78: value 1u -> 10p
- C79: value 10u -> 0.1u
- C84: value 10p -> 10u; device my_rcl:C-1608 -> my_rcl:C-2012
- C9: value 22p -> 560p; device my_rcl:C-1005RF -> my_rcl:C-1608
- D2: value LED -> LOCK
- D3: value LOCK -> LED
- DR1, DR2, DR3, DR4: value HOLE-3.2-CON -> HOLE-3.2C; device my_connector:HOLE-3.2-CON -> my_connector:HOLE-3.2C
- FB6: device my_rcl:FB-2012 -> my_rcl:FB-2012-FB
- IC15: value TAR5SB33 -> TLV431; device my_ic:TAR5SB33 -> my_ic:TL431-SC59
- IC16: value STM32G431K -> TAR5SB33; device my_ic:STM32G431KB -> my_ic:TAR5SB33
- IC3: value STW81200 -> LMX2572; device my_ic:STW81200 -> my_ic:LMX2572
- IC4: value ADL5611 -> SKY65017
- L2: value 47nH -> 100nH; device my_rcl:L-1005RF -> my_rcl:L-1608
- L3: value 47nH -> 33nH; device my_rcl:L-1608 -> my_rcl:L-1005RF
- R3: value 220 -> 1k
- R39, R40: value 1.5k -> 5.1k
- R41: value 1k -> 10k
- R42: value 1k -> 3.6k
- R43: value 10k -> 1k
- R45: value 39 -> 10k
- R46: value 39 -> 1k
- R49, R50: value 5.1k -> 39
- R5: value 150 -> 330
- X1: value 25MHz -> 48MHz
- renumbered X3 to X2
Connections:
- removed net N$31: IC3.HW_PD, J1.2
- removed net N$82: ATT1.SIG2, C25.2
- removed net VIN_PLL: C45.1, C51.1, C57.1, C62.1, FB1.2, IC3.VIN_LDO_4V5, IC3.VIN_LDO_REF, IC3.VIN_LDO_RF_DIG, IC3.VIN_LDO_VCO
- removed net VREG_4V5: C1.1, C2.1, C3.1, C4.1, C5.2, IC3.VCC_CPOUT, IC3.VCC_RFOUT, IC3.VCC_VCO_CORE, IC3.VREG_4V5
- removed net VREG_DIG: C21.2, C24.2, IC3.VDD_DSM_NDIV, IC3.VREG_DIG
- removed net VREG_REF: C19.1, C23.1, IC3.VDD_PFD, IC3.VREG_REF
- removed net VREG_RF: C16.1, C17.1, IC3.VREG_RF
- removed net VREG_VCO: C6.2, C7.1, C8.1, IC3.VDD_CP, IC3.VREG_VCO
- new net N$55: C4.1, IC3.OSCINM
- new net N$88: C3.1, IC3.OSCINP
- new net N$89: C12.1, IC3.VREFVCO
- new net N$90: C11.1, IC3.VREGVCO
- new net N$91: C6.1, IC3.VBIASVCO
- new net N$92: C8.1, IC3.VREGIN
- new net N$93: C17.1, IC3.VBIASVCO2
- new net PLL_EN: IC3.CE, R3.1
- new net VCC_PLL: C19.1, C20.1, C23.1, C24.1, C25.1, C27.1, C28.1, C85.1, C87.1, FB1.1, IC17.VOUT, IC3.VCCBUF, IC3.VCCCP, IC3.VCCDIG, IC3.VCCMASH, IC3.VCCVCO, IC3.VCCVCO2, R3.2
- net +3V3: now also C68.1, C72.1, C84.1, IC16.VOUT; no longer C73.1, C77.1, C87.1, IC15.VOUT
- net +3V3D: now also C77.1, C80.1, C83.1, IC18.VDDA, IC18.VDD_1, IC18.VDD_2; no longer C82.1, C88.1, C89.1, FB7.1, IC16.VDDA, IC16.VDD_1, IC16.VDD_2
- net +5V: now also C47.1, C52.1, C67.1, C70.1, C71.1, C73.1, C74.1, IC16.CONTROL, IC16.VIN, IC17.CONTROL, IC17.VIN, R41.2; no longer C50.1, C56.1, C72.1, C75.1, C76.1, C78.1, FB1.1, IC15.CONTROL, IC15.VIN
- net ADC_IN: now also C60.2, IC18.PA2; no longer C65.2, IC16.PA2
- net ADC_IP: now also C61.1, IC18.PA3; no longer C66.1, IC16.PA3
- net ADC_QN: now also C62.2, IC18.PA0; no longer C67.2, IC16.PA0
- net ADC_QP: now also C63.1, IC18.PA1; no longer C68.1, IC16.PA1
- net AMP_IN: now also C41.2, L9.2; no longer C43.2, L10.2
- net AMP_IP: now also C41.1, L8.2; no longer C43.1, L9.2
- net AMP_QN: now also C42.2, L11.2; no longer C44.2, L12.2
- net AMP_QP: now also C42.1, L10.2; no longer C44.1, L11.2
- net FILTER_IN: now also C26.2; no longer C30.2
- net FIL_SW1: now also IC18.PB5; no longer IC16.PB5
- net FIL_SW2: now also IC18.PB4; no longer IC16.PB4
- net FIL_SW3: now also IC18.PA9; no longer IC16.PA9
- net FIL_SW4: now also IC18.PA8; no longer IC16.PA8
- net GND: now also C24.2, C25.2, C28.2, C43.2, C44.2, C6.2, C60.1, C62.1, C65.2, C67.2, C9.2, D3.K, DR1.HT, DR2.HT, DR3.HT, DR4.HT, IC16.GND, IC17.GND, IC18.VSSA, IC18.VSS_1, IC18.VSS_2, IC3.GND@1, IC3.GND@10, IC3.GND@2, IC3.GND@3, IC3.GND@4, IC3.GND@5, IC3.GND@6, IC3.GND@7, IC3.GND@8, IC3.GND@9, IC3.RAMPCLK, IC3.RAMPDIR, IC3.SYNC, IC3.SYSRELREQ, R44.1, R45.1, R51.1, R52.1, TP9.1; no longer ATT1.GND, C10.2, C21.1, C24.1, C3.2, C60.2, C62.2, C65.1, C67.1, C88.2, C89.2, D2.K, IC16.VSSA, IC16.VSS_1, IC16.VSS_2, IC3.EXTVCO_INN, IC3.EXTVCO_INP, IC3.GND, IC3.PDRF1, IC3.PDRF2, IC3.TEST_SE, J1.1, R41.1, R43.1, R49.1, R50.1
- net N$1: now also C14.1; no longer C15.1
- net N$10: now also C40.1, L10.1, L6.2; no longer C42.1, L11.1, L7.2
- net N$11: now also C40.2, L11.1, L7.2; no longer C42.2, L12.1, L8.2
- net N$12: now also C16.1, IC3.VREFVCO2; no longer C12.1, IC3.VR
- net N$13: now also C82.1, IC17.BYPASS; no longer C5.1, IC3.CBYP_4V5
- net N$14: now also L2.2, L3.1; no longer C27.1, IC3.REF_CLKN
- net N$15: now also IC15.REF, R41.1, R42.2; no longer C6.1, IC3.CBYP
- net N$16: now also IC15.OUT, R43.1; no longer C29.1, IC3.REF_CLKP
- net N$17: now also C34.1; no longer C36.1
- net N$18: now also C36.1; no longer C38.1
- net N$19: now also IC18.PA5, R47.1; no longer IC16.PA5, R45.1
- net N$2: now also C10.2; no longer C14.2
- net N$20: now also C35.1; no longer C37.1
- net N$21: now also C3.2; no longer C29.2
- net N$22: now also C81.1, IC16.BYPASS; no longer C83.1, IC15.BYPASS
- net N$23: now also L1.2; no longer L2.2
- net N$24: now also IC18.PA6, R48.1; no longer IC16.PA6, R46.1
- net N$25: now also IC18.PA7, R49.1; no longer IC16.PA7, R47.1
- net N$26: now also C22.2; no longer C26.2
- net N$27: now also IC18.PB0, R50.1; no longer IC16.PB0, R48.1
- net N$28: now also D3.A, R46.2; no longer D2.A, R44.2
- net N$29: now also R52.2; no longer R50.2
- net N$3: now also C39.1, L4.2, L8.1; no longer C41.1, L5.2, L9.1
- net N$30: now also R51.2; no longer R49.2
- net N$32: now also C29.2, C37.1, L4.1; no longer C31.2, C39.1, L5.1
- net N$33: now also C30.2, C37.2, L5.1; no longer C32.2, C39.2, L6.1
- net N$36: now also R43.2; no longer R41.2
- net N$37: now also D2.K, R44.2; no longer D3.K, R42.2
- net N$39: now also C15.1; no longer C18.1
- net N$4: now also C35.2; no longer C37.2
- net N$40: now also C15.2; no longer C18.2
- net N$41: now also C26.1; no longer C30.1
- net N$42: now also C5.2; no longer C9.2
- net N$43: now also C14.2; no longer C15.2
- net N$44: now also C18.1; no longer C22.1
- net N$5: now also C13.1, IC3.VBIASVARAC; no longer C11.1, R3.2, R4.1
- net N$56: now also C33.2; no longer C35.2
- net N$57: now also C18.2; no longer C22.2
- net N$58: now also C29.1; no longer C31.1
- net N$59: now also C30.1; no longer C32.1
- net N$6: now also C39.2, L5.2, L9.1; no longer C41.2, L10.1, L6.2
- net N$60: now also C31.1; no longer C33.1
- net N$61: now also C32.1; no longer C34.1
- net N$7: now also C31.2, C38.1, L6.1; no longer C33.2, C40.1, L7.1
- net N$70: now also C76.1; no longer C81.1
- net N$71: now also C75.1, IC18.PF0/OSC_IN; no longer C80.1, IC16.PF0/OSC_IN
- net N$72: now also C78.1, IC18.PF1_OSC_OUT; no longer C84.1, IC16.PF1_OSC_OUT
- net N$8: now also C33.1; no longer C35.1
- net N$9: now also C32.2, C38.2, L7.1; no longer C34.2, C40.2, L8.1
- net PGA_SW: now also IC18.PA4, R46.1; no longer IC16.PA4, R44.1
- net PLL_ICP: now also C10.1, C9.1, IC3.CPOUT; no longer C13.1, C14.1, IC3.ICP
- net PLL_OUT: now also C21.2; no longer ATT1.SIG1
- net PLL_OUT1N: now also C22.1, IC3.RFOUTAM; no longer C26.1, IC3.REF2_OUTN
- net PLL_OUT1P: now also C21.1, IC3.RFOUTAP; no longer C25.1, IC3.REF2_OUTP
- net PLL_OUT2N: now also C36.2, IC3.RFOUTBM; no longer C38.2, IC3.REF1_OUTN
- net PLL_OUT2P: now also C34.2, IC3.RFOUTBP; no longer C36.2, IC3.REF1_OUTP
- net PLL_SPI_CS: now also IC3.CSB, R50.2; no longer IC3.LE, R48.2
- net PLL_SPI_MISO: now also D2.A, IC3.MUXOUT, R48.2; no longer D3.A, IC3.SDO, R46.2
- net PLL_SPI_MOSI: now also R49.2; no longer R47.2
- net PLL_SPI_SCK: now also R47.2; no longer R45.2
- net PLL_VCTRL: now also C7.1, IC3.VTUNE, R4.1; no longer C10.1, IC3.VCTRL, R3.1
- net RFIN_SW1: now also IC18.PB6; no longer IC16.PB6
- net RFIN_SW2: now also IC18.PB7; no longer IC16.PB7
- net RF_IN: now also C5.1, L1.1; no longer C9.1, L2.1
- net ST_BOOT0: now also IC18.BOOT0, R45.2; no longer IC16.BOOT0, R43.2
- net ST_NRST: now also C79.1, IC18.NRST; no longer C85.1, IC16.NRST
- net SWCLK: now also IC18.PA14/SWCLK; no longer IC16.PA14/SWCLK
- net SWDIO: now also IC18.PA13/SWDIO; no longer IC16.PA13/SWDIO
- net UART_RX: now also IC18.PA15; no longer IC16.PA15
- net UART_TX: now also IC18.PB3; no longer IC16.PB3
- net USB_DM: now also IC18.PA11; no longer IC16.PA11
- net USB_DP: now also IC18.PA12; no longer IC16.PA12
- net VCC_HFAMP: now also C44.1, C49.1, C54.1, L2.1; no longer C47.1, C53.1, C59.1, L3.1
- net VCC_MIX: now also C43.1, C48.1, C53.1, C57.1, C59.1, C66.1; no longer C46.1, C52.1, C58.1, C63.1, C69.1, C71.1
- net VCC_OSC: now also C1.1, C2.1, FB1.2; no longer C20.1, C79.1, FB7.2
- net VCC_RFSW1: now also C45.1, C50.1, FB4.2; no longer C49.1, C61.1, FB5.2
- net VCC_RFSW2: now also C46.1, C51.1, C56.1, C58.1, FB5.2; no longer C48.1, C54.1, C60.1, FB4.2
- net VCOM: now also C65.1, C69.1; no longer C70.1, C74.1
Other:
- moved on the sheet: C1, C10, C11, C12, C13, C14, C15, C16, C17, C18, C19, C2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
